File: VladMantaAfterActiveTestOpenLine/Eagle/Schematic/Atmega32A.brd (EAGLE design)
At the start: 75.9 x 80 mm, 17 parts, among them IC1 MEGA32-P, IC2 7805T, J1 AVR_SPI_PROG_5X2PTH2, J2 DCJ0202

Commit message: Update
Parts:
- added LED1: (no value), led:LED5MM
- added R2: (no value), rcl:0207/10
Connections:
- new net N$3: LED1.A, R2.1
- net GND: now also LED1.K
- net VCC: now also R2.2
Routing:
- net N$3: track 0.00 -> 16.5 mm
- net GND: track 230.4 -> 239.6 mm
- net VCC: track 179.0 -> 182.1 mm
Changed lines of the file:
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@@
 <attribute name="MF" value="" x="27.94" y="39.37" size="1.778" layer="27" display="off"/>
 </element>
+<element name="R2" library="rcl" package="0207/10" value="" x="67.31" y="74.93"/>
+<element name="LED1" library="led" package="LED5MM" value="" x="45.72" y="76.2" rot="R90"/>
 </elements>
 <signals>
@@
 <wire x1="26.67" y1="77.47" x2="25.4" y2="76.2" width="0.6096" layer="16"/>
 <wire x1="26.67" y1="77.47" x2="36.068" y2="77.47" width="0.6096" layer="16"/>
-<wire x1="36.068" y1="77.47" x2="36.83" y2="76.708" width="0.6096" layer="16"/>
+<wire x1="36.83" y1="76.708" x2="36.068" y2="77.47" width="0.6096" layer="16"/>
 <wire x1="24.13" y1="77.47" x2="25.4" y2="77.47" width="0.6096" layer="16"/>
 <wire x1="25.4" y1="77.47" x2="26.67" y2="77.47" width="0.6096" layer="16"/>
@@
 <wire x1="24.6888" y1="37.3888" x2="25.4" y2="38.1" width="0.6096" layer="16"/>
 <wire x1="25.4" y1="77.47" x2="25.4" y2="76.2" width="0.6096" layer="16"/>
+<contactref element="LED1" pad="K"/>
+<wire x1="37.592" y1="77.47" x2="36.83" y2="76.708" width="0.6096" layer="16"/>
+<wire x1="45.72" y1="77.47" x2="37.592" y2="77.47" width="0.6096" layer="16"/>
 <wire x1="7.62" y1="66.04" x2="5.08" y2="66.04" width="0" layer="19" extent="1-1"/>
 </signal>
@@
 <wire x1="72.39" y1="38.1" x2="73.66" y2="39.37" width="0.6096" layer="16"/>
 <wire x1="73.66" y1="39.37" x2="73.66" y2="69.85" width="0.6096" layer="16"/>
-<wire x1="73.66" y1="69.85" x2="71.12" y2="72.39" width="0.6096" layer="16"/>
+<wire x1="71.12" y1="72.39" x2="73.66" y2="69.85" width="0.6096" layer="16"/>
 <wire x1="71.12" y1="72.39" x2="37.592" y2="72.39" width="0.6096" layer="16"/>
 <wire x1="37.592" y1="72.39" x2="36.83" y2="73.152" width="0.6096" layer="16"/>
@@
 <wire x1="21.59" y1="39.37" x2="39.37" y2="39.37" width="0.6096" layer="16"/>
 <wire x1="39.37" y1="39.37" x2="40.64" y2="40.64" width="0.6096" layer="16"/>
+<contactref element="R2" pad="2"/>
+<wire x1="72.39" y1="74.93" x2="72.39" y2="73.66" width="0.6096" layer="16"/>
+<wire x1="72.39" y1="73.66" x2="71.12" y2="72.39" width="0.6096" layer="16"/>
 </signal>
 <signal name="N$7">
@@
 <wire x1="24.4094" y1="41.6306" x2="24.13" y2="41.91" width="0.6096" layer="16"/>
 </signal>
+<signal name="N$3">
+<contactref element="R2" pad="1"/>
+<contactref element="LED1" pad="A"/>
+<wire x1="45.72" y1="74.93" x2="62.23" y2="74.93" width="0.6096" layer="16"/>
+</signal>
 </signals>
