File: VladMantaAfterActiveTestOpenLine/Eagle/Schematic/Atmega32A.sch (EAGLE design)
At the start: 17 parts, among them IC1 MEGA32-P, IC2 7805T, J1 AVR_SPI_PROG_5X2PTH2, J2 DCJ0202

Commit message: Update
Parts:
- added LED1: (no value), led:LED5MM
- added R2: (no value), rcl:R-EU_0207/10
Connections:
- new net N$3: LED1.A, R2.1
- net GND: now also LED1.C
- net VCC: now also R2.2
Changed lines of the file:
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@@
 <part name="S1" library="switch-omron" deviceset="10-XX" device=""/>
 <part name="GND4" library="supply1" deviceset="GND" device=""/>
+<part name="R2" library="rcl" deviceset="R-EU_" device="0207/10"/>
+<part name="P+5" library="supply1" deviceset="VCC" device=""/>
+<part name="LED1" library="led" deviceset="LED" device="5MM"/>
+<part name="GND5" library="supply1" deviceset="GND" device=""/>
 </parts>
 <sheets>
@@
 <instance part="S1" gate="1" x="38.1" y="25.4"/>
 <instance part="GND4" gate="1" x="40.64" y="12.7"/>
+<instance part="R2" gate="G$1" x="-43.18" y="53.34" rot="R90"/>
+<instance part="P+5" gate="VCC" x="-43.18" y="63.5"/>
+<instance part="LED1" gate="G$1" x="-43.18" y="43.18"/>
+<instance part="GND5" gate="1" x="-43.18" y="33.02"/>
 </instances>
 <busses>
@@
 <junction x="40.64" y="17.78"/>
 </segment>
+<segment>
+<pinref part="LED1" gate="G$1" pin="C"/>
+<pinref part="GND5" gate="1" pin="GND"/>
+<wire x1="-43.18" y1="38.1" x2="-43.18" y2="35.56" width="0.1524" layer="91"/>
+</segment>
 </net>
 <net name="N$4" class="0">
@@
 <wire x1="12.7" y1="63.5" x2="12.7" y2="76.2" width="0.1524" layer="91"/>
 </segment>
+<segment>
+<pinref part="P+5" gate="VCC" pin="VCC"/>
+<pinref part="R2" gate="G$1" pin="2"/>
+<wire x1="-43.18" y1="60.96" x2="-43.18" y2="58.42" width="0.1524" layer="91"/>
+</segment>
 </net>
 <net name="N$7" class="0">
@@
 </segment>
 </net>
+<net name="N$3" class="0">
+<segment>
+<pinref part="R2" gate="G$1" pin="1"/>
+<pinref part="LED1" gate="G$1" pin="A"/>
+<wire x1="-43.18" y1="48.26" x2="-43.18" y2="45.72" width="0.1524" layer="91"/>
+</segment>
+</net>
